File: GPSDO/GPSDO.kicad_sch (KiCad schematic)
At the start: 86 parts, among them IC7 74HC14, J1 Conn_01x01_Pin, J2 SolderJumper_3_Open, J3 SolderJumper_2_Open, K1 Conn_01x04, K2 Conn_01x01_Pin, K3 Conn_01x02, K4 Conn_Coaxial, K5 Jumper_3_Open, K6 Conn_Coaxial, K7 Conn_01x02, K8 Conn_02x03_Odd_Even, K9 Conn_Coaxial, SW1 SW_Nidec_CAS-120A1, U1 LM7805_TO220, U2 DAC8571IDGK, U3 Pico, U4 AD8620, U5 74LVC2G86

Commit message: Changed VCC network, added ICS501 frequency multiplier
Parts:
- removed C24, C25, C26: 100n, Capacitor_SMD:C_1210_3225Metric_Pad1.33x2.70mm_HandSolder, symbol Device:C
- removed J1, TP1, TP2, TP4, TP5: Conn_01x01_Pin, TestPoint:TestPoint_Pad_D1.0mm, symbol Connector:Conn_01x01_Pin
- removed K8: Conn_02x03_Odd_Even, Connector_IDC:IDC-Header_2x03_P2.54mm_Vertical, symbol Connector_Generic:Conn_02x03_Odd_Even
- removed L4, L6: 10µ, Inductor_SMD:L_Cenker_CKCS6045, symbol Device:L
- removed SW1: SW_Nidec_CAS-120A1, Button_Switch_THT:SW_E-Switch_EG1271_SPDT, symbol Switch:SW_Nidec_CAS-120A1
- added C23: C1, symbol Device:C_Polarized
- added C27: C2, symbol Device:C_Polarized
- added C28: C6, Capacitor_SMD:C_1210_3225Metric_Pad1.33x2.70mm_HandSolder, symbol Device:C
- added C29: C8, Capacitor_SMD:C_1210_3225Metric_Pad1.33x2.70mm_HandSolder, symbol Device:C
- added C30: C4, Capacitor_SMD:C_1210_3225Metric_Pad1.33x2.70mm_HandSolder, symbol Device:C
- added C31: C3, Capacitor_SMD:C_1210_3225Metric_Pad1.33x2.70mm_HandSolder, symbol Device:C
- added C32: C7, Capacitor_SMD:C_1210_3225Metric_Pad1.33x2.70mm_HandSolder, symbol Device:C
- added C33: C5, Capacitor_SMD:C_1210_3225Metric_Pad1.33x2.70mm_HandSolder, symbol Device:C
- added C35, C36, C37, C38, C39: 100n, Capacitor_SMD:C_1210_3225Metric_Pad1.33x2.70mm_HandSolder, symbol Device:C
- added D3: D1, symbol Device:D
- added D4: LED, symbol Device:LED
- added J10, J4, J9: Conn_01x02, symbol Connector_Generic:Conn_01x02
- added J11, J5: JP1, symbol Connector_Generic:Conn_02x03_Counter_Clockwise
- added J6, J7: Conn_01x01_Pin, symbol Connector:Conn_01x01_Pin
- added J8: Q2, symbol Connector:Conn_01x01_Pin
- added JP1: Jumper_2_Open, symbol Jumper:Jumper_2_Open
- added K10: Conn_Coaxial, Connector_Coaxial:SMA_Molex_73251-1153_EdgeMount_Horizontal, symbol Connector:Conn_Coaxial
- added L10, L7, L8, L9: 10µ, Inductor_SMD:L_Cenker_CKCS6045, symbol Device:L
- added OCXO1: OCXO, OCXO_example:OSC5A2B02, symbol GPSDO-Components:OSC5A2B02
- added R18: R1, symbol Device:R
- added R19: R2, symbol Device:R
- added R20: R5, symbol Device:R
- added R21: R6, symbol Device:R
- added R3: R3, symbol Device:R
- added R30: R7, symbol Device:R
- added R31: R8, symbol Device:R
- added R32: R9, symbol Device:R
- added R33: R10, symbol Device:R
- added R34: 0, Resistor_SMD:R_1210_3225Metric_Pad1.30x2.65mm_HandSolder, symbol Device:R
- added R35, R36, R37: 10k, Resistor_SMD:R_1210_3225Metric_Pad1.30x2.65mm_HandSolder, symbol Device:R
- added R38, R39: 4.7k, Resistor_SMD:R_1210_3225Metric_Pad1.30x2.65mm_HandSolder, symbol Device:R
- added R40: 50, symbol Device:R
- added R7: R4, symbol Device:R
- added RV3: RV1, Potentiometer_THT:Potentiometer_Bourns_3266Y_Vertical, symbol Device:R_Potentiometer
- added U6, U8: U1, symbol GPSDO-Components:ICS501
- added U7: IC1, Package_TO_SOT_SMD:SOT-223-3_TabPin2, symbol Regulator_Linear:LM7805_TO220
- added U9: CAT24C128, symbol Memory_EEPROM:CAT24C128
- C15: value 0.1u -> 100n
Connections:
- net GND: now also C23.2, C27.2, C28.1, C30.2, C31.2, C35.2, C36.1, C37.1, C38.1, C39.1, J10.2 (Pin_2), J11.3 (Pin_3), J11.4 (Pin_4), J5.3 (Pin_3), J5.4 (Pin_4), J7.1 (Pin_1), J9.2 (Pin_2), JP1.1 (A), K10.2 (Ext), OCXO1.2 (GND), R18.2, R32.2, R7.2, RV3.1, U6.3 (GND), U7.2 (GND), U8.3 (GND), U9.1 (A0), U9.2 (A1), U9.3 (A2), U9.4 (GND)
- net VCC: now also C21.1, C7.1, C8.1, IC1.1 (LD), L2.2, R22.1, U1.3 (VO), U3.40 (VBUS), L10.1, L7.1, L8.1, L9.1; no longer C15.1, IC2.8 (V+), L2.1, R14.1
- net at K9.1 (In), R24.1, R25.1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: now also R28.1, R34.1
- net at C1.1, K1.1 (Pin_1), R12.2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: now also R35.1, R36.1, R37.1, U9.8 (VCC)
- net at OCXO2.3 (Vcont), R16.1, U4.6 (-): now also C22.1
- net at U3.26 (GPIO20): now also R35.2, U9.5 (SDA)
- net at U3.27 (GPIO21): now also R36.2, U9.6 (SCL)
- removed net VCC_1: C21.1, C22.1, IC3.16 (VCC), IC6.16 (VCC), IC7.14 (VCC), R22.1, U5.8 (VCC)
- new net: C36.2, C37.2, IC3.16 (VCC), IC6.16 (VCC), L7.2
- new net: C28.2, OCXO1.1 (10MHz), R19.2
- new net: C23.1, D3.1 (K), U7.1 (VI)
- new net: C27.1, C30.1, C31.1, D4.2 (A), OCXO1.4 (NC), R20.1, R21.1, R3.1, R33.1, RV3.3, U6.2 (VDD), U6.7 (OE), U7.3 (VO)
- new net: C29.1, J9.1 (Pin_1)
- new net: C33.2, R3.2, R7.1, U6.1 (X1/CLK)
- new net: C38.2, IC7.14 (VCC), L9.2
- new net: D3.2 (A), J4.2 (Pin_2)
- new net: R34.2, U8.1 (X1/CLK)
- new net: C35.1, L2.1, R38.2, R39.1, U8.2 (VDD), U8.7 (OE)
- new net: J11.2 (Pin_2), U8.4 (S1)
- new net: R40.1, U8.5 (CLK)
- new net: J11.5 (Pin_5), U8.6 (S0)
- new net: JP1.2 (B), R37.2, U9.7 (WP)
- new net: C15.1, IC2.8 (V+), L10.2, R14.1
- new net: J5.1 (Pin_1), R20.2
- new net: C32.1, C33.1, OCXO1.3 (Vcont)
- new net: D4.1 (K), R18.1
- new net: J10.1 (Pin_1), R30.1
- new net: R30.2, U6.5 (CLK)
- new net: J6.1 (Pin_1), R31.1, R32.1
- new net: R19.1, RV3.2
- new net: C32.2, R31.2
- new net: J11.6 (Pin_6), R39.2
- new net: J5.6 (Pin_6), R21.2
- new net: J5.2 (Pin_2), U6.4 (S1)
- new net: J5.5 (Pin_5), U6.6 (S0)
- new net: C39.2, L8.2, U5.8 (VCC)
- new net: J11.1 (Pin_1), R38.1
- new net: K10.1 (In), R40.2
- new net: C29.2, J8.1 (Pin_1), R33.2
Other:
- note added: "100mA SMD klein"
- note added: "100uH groß https://www.mouser.de/ProductDetail/TDK/SPM7054VC-101M-D?qs=sGAEpiMZZMv126LJFLh8yz4JeXP9OGKgXN2nn20c%2F50%3D"
- note added: "10uH groß https://www.mouser.de/ProductDetail/Monolithic-Power-Systems-MPS/MPL-SE5040-100?qs=sGAEpiMZZMv126LJFLh8yyOx6Bzv8ule8YDMbIBSVtI%3D"
- note added: "20mA SMD klein"
- note added: "25mA SMD klein"
- note added: "50mA SMD klein"
- note added: "7.5V - 9V GND"
- note added: "Barrel-Jack DC connector - prinzipiell egal welcher https://www.mouser.de/ProductDetail/CUI-Devices/PJ-102AH?qs=WyjlAZoYn50Yq4CrVLCXLw%3D%3D"
- note added: "D1 Schottky-Diode https://www.mouser.de/ProductDetail/onsemi-Fairchild/SS24FL?qs=tqW9UTzndZyvT5hdH%2BfSxg%3D%3D"
- note added: "D2 Entstördiode https://www.mouser.de/ProductDetail/Nexperia/PESD5V5H1BSFYL?qs=T3oQrply3y9CfA%2FMHqAcog%3D%3D"
- note added: "EEPROM https://www.mouser.de/ProductDetail/onsemi/CAT24C32WI-GT3?qs=rZgeL6XvLwaTa79VuYkKQA%3D%3D"
- note added: "ICS501 https://www.mouser.de/ProductDetail/Renesas-Electronics/501MLFT?qs=JcGQCygHkIZqmlnfOhnKLQ%3D%3D"
- note added: "Kleinstrom-Induktivitätem 100µH https://www.mouser.de/ProductDetail/TDK/KLZ2012NHR101LTD25?qs=5aG0NVq1C4xezrpiGY6jhA%3D%3D"
- note added: "Kleinstrom-Induktivitäten 10µH https://www.mouser.de/ProductDetail/TDK/KLZ2012MHR100HTD25?qs=5aG0NVq1C4z7XTXkifhyMA%3D%3D"
- note added: "PINOUT OF OCXO DOESN'T MATCH THE ONE ON CIRCUIT"
- note added: "S0"
- note added: "S1"
- note added: "SMD klein"
- note added: "ToDo Patrick: Widerstände vor und hinter die Potis?"
- note added: "Transistor?"
- note removed: "+5V"
- note removed: "100uH https://www.mouser.de/ProductDetail/TDK/SPM7054VC-101M-D?qs=sGAEpiMZZMv126LJFLh8yz4JeXP9OGKgXN2nn20c%2F50%3D"
- note removed: "10uH https://www.mouser.de/ProductDetail/Monolithic-Power-Systems-MPS/MPL-SE5040-100?qs=sGAEpiMZZMv126LJFLh8yyOx6Bzv8ule8YDMbIBSVtI%3D"
- note removed: "Barrel-Jack DC connector https://www.mouser.de/ProductDetail/CUI-Devices/PJ-102AH?qs=WyjlAZoYn50Yq4CrVLCXLw%3D%3D"
- note removed: "Fanout Buffer Board"
- moved on the sheet: C20, C21, C5, C7, C8, D2, IC3C, IC6C, IC7F, L3, U5C

Commit message: added voltage reference to DAC
Parts:
- removed C23: C1, symbol Device:C_Polarized
- removed C27: C2, symbol Device:C_Polarized
- removed C28: C6, Capacitor_SMD:C_1210_3225Metric_Pad1.33x2.70mm_HandSolder, symbol Device:C
- removed C29: C8, Capacitor_SMD:C_1210_3225Metric_Pad1.33x2.70mm_HandSolder, symbol Device:C
- removed C30: C4, Capacitor_SMD:C_1210_3225Metric_Pad1.33x2.70mm_HandSolder, symbol Device:C
- removed C31: C3, Capacitor_SMD:C_1210_3225Metric_Pad1.33x2.70mm_HandSolder, symbol Device:C
- removed C32: C7, Capacitor_SMD:C_1210_3225Metric_Pad1.33x2.70mm_HandSolder, symbol Device:C
- removed C33: C5, Capacitor_SMD:C_1210_3225Metric_Pad1.33x2.70mm_HandSolder, symbol Device:C
- removed D3: D1, symbol Device:D
- removed D4: LED, symbol Device:LED
- removed J10, J4, J9: Conn_01x02, symbol Connector_Generic:Conn_01x02
- removed J5: JP1, symbol Connector_Generic:Conn_02x03_Counter_Clockwise
- removed J6, J7: Conn_01x01_Pin, symbol Connector:Conn_01x01_Pin
- removed J8: Q2, symbol Connector:Conn_01x01_Pin
- removed K2: Conn_01x01_Pin, TestPoint:TestPoint_Loop_D2.50mm_Drill1.85mm, symbol Connector:Conn_01x01_Pin
- removed OCXO1: OCXO, OCXO_example:OSC5A2B02, symbol GPSDO-Components:OSC5A2B02
- removed R21: R6, symbol Device:R
- removed R30: R7, symbol Device:R
- removed R31: R8, symbol Device:R
- removed R32: R9, symbol Device:R
- removed R33: R10, symbol Device:R
- removed R34: 0, Resistor_SMD:R_1210_3225Metric_Pad1.30x2.65mm_HandSolder, symbol Device:R
- removed RV3: RV1, Potentiometer_THT:Potentiometer_Bourns_3266Y_Vertical, symbol Device:R_Potentiometer
- removed U6: U1, symbol GPSDO-Components:ICS501
- removed U7: IC1, Package_TO_SOT_SMD:SOT-223-3_TabPin2, symbol Regulator_Linear:LM7805_TO220
- added C23: 100n, Capacitor_SMD:C_1210_3225Metric_Pad1.33x2.70mm_HandSolder, symbol Device:C
- added K8: Conn_Coaxial, Connector_Coaxial:SMA_Molex_73251-1153_EdgeMount_Horizontal, symbol Connector:Conn_Coaxial
- added U6: LM4040DBZ-4.1, Package_TO_SOT_SMD:SOT-23, symbol Reference_Voltage:LM4040DBZ-4.1
- J11: footprint (none) -> Connector_PinHeader_2.54mm:PinHeader_2x03_P2.54mm_Vertical
- JP1: footprint (none) -> Connector_PinHeader_2.54mm:PinHeader_1x02_P2.54mm_Vertical
- L1, L5: footprint Inductor_SMD:L_Neosid_SM-PIC0612H -> Inductor_SMD:L_0805_2012Metric_Pad1.15x1.40mm_HandSolder
- L10, L2, L7, L8, L9: footprint Inductor_SMD:L_Cenker_CKCS6045 -> Inductor_SMD:L_0805_2012Metric_Pad1.15x1.40mm_HandSolder
- R18: value R1 -> 50; footprint (none) -> Resistor_SMD:R_1210_3225Metric_Pad1.30x2.65mm_HandSolder
- R19: value R2 -> 50; footprint (none) -> Resistor_SMD:R_1210_3225Metric_Pad1.30x2.65mm_HandSolder
- R20: value R5 -> 1k; footprint (none) -> Resistor_SMD:R_1210_3225Metric_Pad1.30x2.65mm_HandSolder
- R3: value R3 -> 100k; footprint (none) -> Resistor_SMD:R_1210_3225Metric_Pad1.30x2.65mm_HandSolder
- R40: footprint (none) -> Resistor_SMD:R_1210_3225Metric_Pad1.30x2.65mm_HandSolder
- R7: value R4 -> 100k; footprint (none) -> Resistor_SMD:R_1210_3225Metric_Pad1.30x2.65mm_HandSolder
- U8, U9: footprint (none) -> Package_SO:SOIC-8_3.9x4.9mm_P1.27mm
Connections:
- net GND: now also K8.2 (Ext), U6.2 (A); no longer R18.2
- net VCC: now also R3.1; no longer IC1.1 (LD)
- net at R2.2: now also K8.1 (In)
- net at R19.2: now also K6.1 (In)
- net at R20.1: now also C13.1, C14.1, L5.1, U4.8 (V+); no longer R3.1
- net at K9.1 (In), R24.1, R25.1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: now also C23.2
- net at R3.2, R7.1: now also U8.1 (X1/CLK), C23.1
- net at R20.2: now also U2.1 (V_{DD}), U2.2 (V_{REF}), U6.1 (K)
- net at R18.1: now also U5.3
- net at R19.1: now also RV1.3, U5.6, U5.7
- net at U3.5 (GPIO3): now also IC1.1 (LD)
- net at K4.1 (In): now also R18.2; no longer U5.3
Other:
- note added: "Leave open if this upconverter is unused or make solder bridge if no DC offset is needed."
- note added: "Only place these if DC offset is needed"
- note removed: "7.5V - 9V GND"
- note removed: "Jumper?"
- note removed: "PINOUT OF OCXO DOESN'T MATCH THE ONE ON CIRCUIT"
- note removed: "S0"
- note removed: "S1"
- note removed: "Transistor?"
- moved on the sheet: C7, K4, K6, R22, R23, U2

Commit message: buffers added + cleanup
Parts:
- added C24, C25, C26: 100n, Capacitor_SMD:C_1210_3225Metric_Pad1.33x2.70mm_HandSolder, symbol Device:C
- added IC4, IC5, IC8: 74HC14, Package_SO:SOIC-14_3.9x8.7mm_P1.27mm, symbol 74xx:74HC14
- added L11, L4, L6: 10µ, Inductor_SMD:L_0805_2012Metric_Pad1.15x1.40mm_HandSolder, symbol Device:L
- added R21, R30, R31, R32, R33, R34, R41, R42, R43: 240, Resistor_SMD:R_1210_3225Metric_Pad1.30x2.65mm_HandSolder, symbol Device:R
- R18, R19, R40: value 50 -> 240
Connections:
- net GND: now also C24.1, C25.1, C26.1, IC4.7 (GND), IC5.7 (GND), IC8.7 (GND)
- net VCC: now also L11.1, L4.1, L6.1
- net at U8.5 (CLK): now also IC8.13, IC8.3, IC8.5, IC8.9; no longer R40.1
- net at U5.3: now also IC4.13, IC4.3, IC4.5, IC4.9; no longer R18.1
- net at R19.1, RV1.3, U5.6: now also K6.1 (In), R33.1, R34.1, R41.1; no longer U5.7
- net at R19.2: now also IC5.6; no longer K6.1 (In)
- net at R40.2: now also IC8.8; no longer K10.1 (In)
- net at R18.2: now also IC8.6; no longer K4.1 (In)
- new net: C26.2, IC8.14 (VCC), L11.2
- new net: IC5.13, IC5.3, IC5.5, IC5.9, U5.7
- new net: IC5.4, R34.2
- new net: IC4.6, R21.2
- new net: K4.1 (In), R21.1, R30.1, R31.1, R32.1
- new net: IC4.8, R30.2
- new net: R18.1, R40.1, R42.1, R43.1
- new net: IC8.12, R43.2
- new net: C25.2, IC5.14 (VCC), L6.2
- new net: IC8.4, R42.2
- new net: C24.2, IC4.14 (VCC), L4.2
- new net: IC4.4, R31.2
- new net: IC4.12, R32.2
- new net: IC5.8, R33.2
- new net: IC5.12, R41.2
Other:
- moved on the sheet: C1, C10, C11, C12, C13, C14, C15, C16, C17, C18, C19, C2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
