File: GPSDO_DIP/GPSDO_DIP/GPSDO_DIP.kicad_pcb (KiCad board)
At the start: 2 copper layers, 126.1 x 87.1 mm, 86 parts, among them IC2 74HC14, K1 Conn_01x04, K2 Conn_Coaxial, K3 Conn_01x02, K4 Jumper_3_Open, K5 Conn_01x02, K9 Conn_Coaxial, U1 Pico, U10 U1, U11 74HC14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

Commit message: added mounting holes & 10MHz SMA-port, cleaned up labels a bit
Parts:
- added K6: Conn_Coaxial, Connector_Coaxial:SMA_Molex_73251-1153_EdgeMount_Horizontal, F.Cu at (138.0, 58.8)
- added REF**: MountingHole_3.2mm_M3_Pad_Via, MountingHole:MountingHole_3.2mm_M3_Pad_Via, F.Cu at (91.8, 15.5)
- added REF**: MountingHole_3.2mm_M3_Pad_Via, MountingHole:MountingHole_3.2mm_M3_Pad_Via, F.Cu at (137.0, 91.2)
- added REF**: MountingHole_3.2mm_M3_Pad_Via, MountingHole:MountingHole_3.2mm_M3_Pad_Via, F.Cu at (22.3, 91.2)
- added REF**: MountingHole_3.2mm_M3_Pad_Via, MountingHole:MountingHole_3.2mm_M3_Pad_Via, F.Cu at (22.3, 15.5)
- moved C1 5.00 mm to (28.0, 17.8)
- moved K3 2.60 mm to (19.6, 41.3)
- moved K1 2.60 mm to (19.6, 22.2)
- moved R3 2.60 mm to (19.5, 34.3)
- moved K5 2.00 mm to (30.4, 77.0)
- moved K2 0.30 mm to (80.8, 14.8)
- moved K9 0.30 mm to (102.7, 14.8)
- moved R2 0.10 mm to (80.8, 20.0)
- renumbered IC1 to U2, IC2 to U3, U10 to U4, U11 to U8, U4 to U9
Routing:
- net Net-(K6-In): track 18.7 -> 30.1 mm
- net GND: track 30.4 -> 34.6 mm, vias 3 -> 14
- net Net-(K1-Pin_2): track 7.12 -> 8.22 mm
- net Net-(U1-GPIO2): track 7.34 -> 8.41 mm
- net Net-(K1-Pin_1): track 59.2 -> 60.3 mm
- net Net-(K1-Pin_3): track 7.12 -> 8.16 mm
- net Net-(D1-A): track 6.93 -> 7.76 mm
Other:
- board text added: "1 PPS in"
- board text added: "10MHz out"
- board text added: "40MHz out"
- board text added: "PC2 PC1"
